File: circuit/circuit.sch (KiCad schematic (older format))
At the start: 6 parts

Commit message: made progress on schematic
Parts:
- added C? (x2): C_30pF, footprints:C_0805_OEM, symbol formula:C_30pF
- added R? (x8): R_100K, footprints:R_0805_OEM, symbol formula:R_100K
- added R? (x8): R_1M, footprints:R_0805_OEM, symbol formula:R_1M
- added R? (x8): R_200, footprints:R_0805_OEM, symbol formula:R_200
- added U? (x8): LMC6484, symbol Amplifier_Operational:LMC6484
- added U? (x8): AD623BRZ, symbol Amplifier_Instrumentation:AD623BRZ
- added U?: AMS1117-5.0, Package_TO_SOT_SMD:SOT-223-3_TabPin2, symbol Regulator_Linear:AMS1117-5.0
- added U?: IDTQS3253, symbol formula:IDTQS3253
- added U?: DRV8834, symbol formula:DRV8834
- added Y?: Crystal_SMD, footprints:Crystal_SMD_FA238, symbol formula:Crystal_SMD
Connections:
- net labels added: battery+, battery-, blue_1, blue_2, blue_3, blue_4, diode_1, diode_2, diode_3, diode_4, diode_5, diode_6, diode_7, diode_9, enable_A, enable_B, red_1, red_2, red_3, red_4, select_0, select_1
- net labels removed: ADC0, ADC5
- wire segments 18 -> 242
Other:
- moved on the sheet: C?, R?, U?

Commit message: more progess git add -A!
Parts:
- removed R? (x8): R_100K, footprints:R_0805_OEM, symbol formula:R_100K
- removed R? (x8): R_200, footprints:R_0805_OEM, symbol formula:R_200
- removed R? (x7): R_1M, footprints:R_0805_OEM, symbol formula:R_1M
- removed U? (x8): AD623BRZ, symbol Amplifier_Instrumentation:AD623BRZ
- removed U? (x7): LMC6484, symbol Amplifier_Operational:LMC6484
- removed U?: IDTQS3253, symbol formula:IDTQS3253
- added C4: C_0.01uF, footprints:C_0805_OEM, symbol formula:C_0.1uF
- added C5: C_2.2uF, footprints:C_0603_1608Metric, symbol formula:C_2.2uF
- added D1, D2: LED_0805, footprints:LED_0805_OEM, symbol formula:LED_0805
- added F1: F_3.15A_300V, footprints:Fuse_TE7_Littelfuse-807Series, symbol formula:F_3.15A_300V
- added J1: Conn_01x14_Female, symbol Connector:Conn_01x14_Female
- added J3: Conn_02x03_Odd_Even, symbol Connector_Generic:Conn_02x03_Odd_Even
- added R1, R2, R21, R22, R23, R24, R3: R_1M, footprints:R_0805_OEM, symbol formula:R_1M
- added R10, R12, R26, R28, R30, R32, R6, R8: R_10K, footprints:R_0805_OEM, symbol formula:R_10K
- added R11, R13, R14, R15, R16, R25, R27, R29, R31, R33, R34, R35, R36, R5, R7, R9: R_100K, footprints:R_0805_OEM, symbol formula:R_100K
- added R17, R18, R19, R20, R37, R38, R39, R40, R44, R45, R46: R_200, footprints:R_0805_OEM, symbol formula:R_200
- added R41: R_47K, footprints:R_0805_OEM, symbol formula:R_1K
- added unit 5 of U1
- added unit 2 of U1
- added unit 3 of U1
- added unit 4 of U1
- added U12, U13, U5, U6: LM358DT, Housings_SOIC:SO-8_5.3x6.2mm_Pitch1.27mm, symbol formula:LM358DT
- added U14: SN74LV4052APWR, symbol formula:SN74LV4052APWR
- added U2: LMC6484, symbol Amplifier_Operational:LMC6484
- U1: renamed from U?; footprint (none) -> Housings_SOIC:SOIC-14_3.9x8.7mm_Pitch1.27mm
- U7: renamed from U?; value AMS1117-5.0 -> L78M05CDT-TR
- gave numbers to parts that had none: 11
Connections:
- net labels added: a_out, b_out, diode_8, issues, led_D1, led_D2, led_D3, motorA+, motorA-, motorA_DIR, motorA_PWM, motorB+, motorB-, motorB_DIR, motorB_PWM, p_led
- net labels removed: diode_9, enable_A, enable_B
- wire segments 242 -> 243
- no-connect marks 0 -> 6
Other:
- note added: "AUXILIARY HARDWARE"
- note added: "BLUE DIODE CIRCUIT"
- note added: "CONNECTORS"
- note added: "MAIN"
- note added: "MOTOR DRIVER"
- note added: "NEW CIRCUIT"
- note added: "ORIGINAL CIRCUIT"
- note added: "PINOUT"
- note added: "POWER"
- note added: "POWER REGULATORS\n"
- note added: "PROGRAMMING\n"
- note added: "RED DIODE CIRCUIT"
- moved on the sheet: C1, C2, C3, C6, R4, R43, U15, U16, U1A, U7, Y1

Commit message: finished schematic for main board
Parts:
- removed F1: F_3.15A_300V, footprints:Fuse_TE7_Littelfuse-807Series, symbol formula:F_3.15A_300V
- removed J1: Conn_01x14_Female, symbol Connector:Conn_01x14_Female
- removed R1, R2, R21, R22, R23: R_1M, footprints:R_0805_OEM, symbol formula:R_1M
- removed R10, R26, R28, R30, R6, R8: R_10K, footprints:R_0805_OEM, symbol formula:R_10K
- removed R13, R14, R15, R25, R27, R29, R33, R34, R35, R5, R7: R_100K, footprints:R_0805_OEM, symbol formula:R_100K
- removed R17, R18, R19, R37, R38, R39: R_200, footprints:R_0805_OEM, symbol formula:R_200
- removed unit 3 of U1
- removed U12, U5: LM358DT, Housings_SOIC:SO-8_5.3x6.2mm_Pitch1.27mm, symbol formula:LM358DT
- removed unit 1 of U13
- removed unit 5 of U2
- removed unit 2 of U2
- removed unit 3 of U2
- removed unit 4 of U2
- removed unit 1 of U6
- added C1: C_0.1uF, footprints:C_0805_OEM, symbol formula:C_0.1uF
- added F?: Fuse_2A, Resistors_SMD:R_0402, symbol Device:Fuse
- added J1: Conn_01x20_Female, footprints:Pin_Header_Straight_2x10, symbol Connector:Conn_01x20_Female
- added R11, R22: R_200, footprints:R_0805_OEM, symbol formula:R_200
- added R14: R_1M, footprints:R_0805_OEM, symbol formula:R_1M
- added R16, R20, R6: R_100K, footprints:R_0805_OEM, symbol formula:R_100K
- added R17, R7: R_10K, footprints:R_0805_OEM, symbol formula:R_10K
- added U3: LM358DT, Housings_SOIC:SO-8_5.3x6.2mm_Pitch1.27mm, symbol formula:LM358DT
- added U6: SN74LV4052APWR, Housings_SSOP:TSSOP-16_4.4x5mm_Pitch0.65mm, symbol formula:SN74LV4052APWR
- J2: renamed from J3; footprint (none) -> footprints:Pin_Header_Straight_2x03
- U4: renamed from U7; footprint Package_TO_SOT_SMD:SOT-223-3_TabPin2 -> footprints:L78M05CDT-TR
- U5: renamed from U14; footprint (none) -> Housings_SSOP:TSSOP-16_4.4x5mm_Pitch0.65mm
- U7: renamed from U15; footprint (none) -> footprints:DRV8834PWP
- renumbered C1 to C2, C2 to C3, C3 to C4, C4 to C5, C5 to C6, C6 to C7, R44 to R1, R20 to R10, R45 to R12, R46 to R13, R24 to R15, R31 to R18, R32 to R19, R4 to R2, R36 to R21, R40 to R23, R41 to R24, R42 to R25, R43 to R26, R11 to R4, R12 to R5, R16 to R8, U2 to U1, U6 to U2, U13 to U2, U16 to U8
Connections:
- net labels added: blue_5, blue_6, blue_7, blue_8, blue_inA, blue_inB, blue_outA, blue_outB, red_5, red_6, red_7, red_8, red_inA, red_inB, red_out1A, red_outA, red_outB, select_0A, select_0B, select_1A, select_1B
- net labels removed: a_out, b_out, diode_1, diode_2, diode_3, diode_4, diode_5, diode_6, diode_7, diode_8, led_D2, led_D3, select_0, select_1
- wire segments 243 -> 178
- no-connect marks 6 -> 4
Other:
- note added: "LEDS\n"
- note added: "SUPPORTING IMAGES"
- moved on the sheet: D1, D2, R1, R12, R13

Commit message: finished schematic for main board
Parts:
- added R1, R2: R_10K, footprints:R_0805_OEM, symbol formula:R_10K
- added U2: LIS3DHTR, footprints:LIS3DHTR, symbol formula:LIS3DHTR
- added U6: LM3480, TO_SOT_Packages_SMD:SOT-23-3-Lead_TabPin2, symbol formula:LM3480
- U10: renamed from U8; footprint Package_DIP:DIP-28_W7.62mm -> footprints:ATMEGA_328PB_CONN
- gave numbers to parts that had none: 1
- renumbered R8 to R10, R9 to R11, R10 to R12, R11 to R13, R12 to R14, R13 to R15, R14 to R16, R15 to R17, R16 to R18, R17 to R19, R18 to R20, R19 to R21, R20 to R22, R21 to R23, R22 to R24, R23 to R25, R24 to R26, R25 to R27, R26 to R28, R1 to R3, R2 to R4, R3 to R5, R4 to R6, R5 to R7, R6 to R8, R7 to R9, U2 to U3, U3 to U4, U4 to U5, U5 to U7, U6 to U8, U7 to U9
Connections:
- net labels added: 3.3V, SCL, SDA
- net labels removed: red_out1A
- wire segments 178 -> 201
- no-connect marks 4 -> 8
Other:
- note added: "ACCELEROMETER"
- moved on the sheet: D1, D2, R14, R15, U5

Commit message: finished schematic for main board
Parts:
- U6: footprint TO_SOT_Packages_SMD:SOT-23-3-Lead_TabPin2 -> TO_SOT_Packages_SMD:SOT-23
Changed lines of the file:
@@
 	-1   0    0    -1
 $EndComp
-Text Label 950  2850 0    50   ~ 0
+Text Label 950  3250 0    50   ~ 0
 red_4
-Text Label 950  2950 0    50   ~ 0
+Text Label 950  3350 0    50   ~ 0
 red_3
-Text Label 950  3050 0    50   ~ 0
+Text Label 950  3450 0    50   ~ 0
 red_2
-Text Label 950  3150 0    50   ~ 0
+Text Label 950  3550 0    50   ~ 0
 red_1
 Text Label 950  2450 0    50   ~ 0
@@
 Text Label 950  2750 0    50   ~ 0
 red_5
-Text Label 950  3550 0    50   ~ 0
+Text Label 950  3150 0    50   ~ 0
 blue_5
-Text Label 950  3450 0    50   ~ 0
+Text Label 950  3050 0    50   ~ 0
 blue_6
-Text Label 950  3350 0    50   ~ 0
+Text Label 950  2950 0    50   ~ 0
 blue_7
-Text Label 950  3250 0    50   ~ 0
+Text Label 950  2850 0    50   ~ 0
 blue_8
 $Comp
@@
 F 0 "U6" H 5750 1542 50  0000 C CNN
 F 1 "LM3480" H 5750 1451 50  0000 C CNN
-F 2 "TO_SOT_Packages_SMD:SOT-23-3-Lead_TabPin2" H 5700 1500 50  0001 C CNN
+F 2 "TO_SOT_Packages_SMD:SOT-23" H 5700 1500 50  0001 C CNN
 F 3 "http://www.ti.com/lit/ds/symlink/lm3480.pdf" H 5850 1050 50  0001 C CNN
 F 4 "DK" H 5800 1625 60  0001 C CNN "MFN"

Commit message: started on layout. *make crab noise*
Parts:
- added C8: C_0.1uF, footprints:C_0805_OEM, symbol formula:C_0.1uF
- added R29, R30: R_10K, footprints:R_0805_OEM, symbol formula:R_10K
- C5: PurchasingLink https://www.digikey.com/products/en?keywords=478-3352-1-ND -> https://www.digikey.com/product-detail/en/samsung-electro-m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
- C6: footprint footprints:C_0603_1608Metric -> footprints:R_0805_OEM; PurchasingLink https://www.digikey.com/product-detail/en/yageo/CC0603KRX5R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 -> https://www.digikey.com/product-detail/en/taiyo-yuden/EMK21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
- F1: value Fuse_2A -> Fuse_1A
Connections:
- wire segments 201 -> 210
- no-connect marks 8 -> 7
Changed lines of the file:
@@
 F 0 "C6" H 15415 6396 50  0000 L CNN
 F 1 "C_2.2uF" H 15415 6305 50  0000 L CNN
-F 2 "footprints:C_0603_1608Metric" H 15338 6200 50  0001 C CNN
-F 3 "http://www.yageo.com/documents/recent/UPY-GPHC_X5R_4V-to-50V_25.pdf" H 15325 6450 50  0001 C CNN
+F 2 "footprints:R_0805_OEM" H 15338 6200 50  0001 C CNN
+F 3 "" H 15325 6450 50  0001 C CNN
 F 4 "DK" H 15300 6350 60  0001 C CNN "MFN"
 F 5 "311-1451-1-ND" H 15300 6350 60  0001 C CNN "MPN"
-F 6 "https://www.digikey.com/product-detail/en/yageo/CC0603KRX5R6BB225/311-1451-1-ND/2833757" H 15725 6850 60  0001 C CNN "PurchasingLink"
+F 6 "https://www.digikey.com/product-detail/en/taiyo-yuden/EMK212BJ225KGHT/587-3323-1-ND/4157368" H 15725 6850 60  0001 C CNN "PurchasingLink"
 	1    15300 6350
 	1    0    0    -1
@@
 F 1 "C_0.01uF" V 15050 6400 50  0000 C CNN
 F 2 "footprints:C_0805_OEM" H 15038 6250 50  0001 C CNN
-F 3 "http://datasheets.avx.com/X7RDielectric.pdf" H 15025 6500 50  0001 C CNN
+F 3 "" H 15025 6500 50  0001 C CNN
 F 4 "DK" H 15000 6400 60  0001 C CNN "MFN"
 F 5 "478-3352-1-ND" H 15000 6400 60  0001 C CNN "MPN"
-F 6 "https://www.digikey.com/products/en?keywords=478-3352-1-ND" H 15425 6900 60  0001 C CNN "PurchasingLink"
+F 6 "https://www.digikey.com/product-detail/en/samsung-electro-mechanics/CL21B103KBCSFNC/1276-2439-1-ND/3890525" H 15425 6900 60  0001 C CNN "PurchasingLink"
 	1    15000 6400
 	0    1    1    0
@@
 P 1600 1700
 F 0 "F1" H 1660 1746 50  0000 L CNN
-F 1 "Fuse_2A" H 1660 1655 50  0000 L CNN
+F 1 "Fuse_1A" H 1660 1655 50  0000 L CNN
 F 2 "Resistors_SMD:R_0402" V 1530 1700 50  0001 C CNN
 F 3 "https://industrial.panasonic.com/cdbs/www-data/pdf/AFA0000/AFA0000C7.pdf" H 1600 1700 50  0001 C CNN
@@
 Wire Wire Line
 	1350 10250 1350 10350
-$Comp
-L power:VCC #PWR05
-U 1 1 5BE22060
-P 1350 10350
-F 0 "#PWR05" H 1350 10200 50  0001 C CNN
-F 1 "VCC" H 1368 10523 50  0000 C CNN
-F 2 "" H 1350 10350 50  0001 C CNN
-F 3 "" H 1350 10350 50  0001 C CNN
-	1    1350 10350
-	-1   0    0    1
-$EndComp
 NoConn ~ 3200 10050
 NoConn ~ 3200 10250
-Wire Wire Line
-	3200 9950 3600 9950
 $Comp
 L power:GND #PWR019
 U 1 1 5BE408C1
-P 3600 10200
-F 0 "#PWR019" H 3600 9950 50  0001 C CNN
-F 1 "GND" H 3605 10027 50  0000 C CNN
-F 2 "" H 3600 10200 50  0001 C CNN
-F 3 "" H 3600 10200 50  0001 C CNN
-	1    3600 10200
+P 3500 10250
+F 0 "#PWR019" H 3500 10000 50  0001 C CNN
+F 1 "GND" H 3505 10077 50  0000 C CNN
+F 2 "" H 3500 10250 50  0001 C CNN
+F 3 "" H 3500 10250 50  0001 C CNN
+	1    3500 10250
 	1    0    0    -1
 $EndComp
-Wire Wire Line
-	3200 10150 3600 10150
-Wire Wire Line
-	3600 10150 3600 10200
-Wire Wire Line
-	3600 9950 3600 10150
-Connection ~ 3600 10150
 NoConn ~ 3200 9850
 NoConn ~ 3200 9550
 NoConn ~ 3200 9650
-NoConn ~ 1350 10150
 $Comp
 L power:GND #PWR04
 U 1 1 5BEB9C0E
-P 1150 10350
-F 0 "#PWR04" H 1150 10100 50  0001 C CNN
-F 1 "GND" H 1155 10177 50  0000 C CNN
-F 2 "" H 1150 10350 50  0001 C CNN
-F 3 "" H 1150 10350 50  0001 C CNN
-	1    1150 10350
+P 800 10200
+F 0 "#PWR04" H 800 9950 50  0001 C CNN
+F 1 "GND" H 805 10027 50  0000 C CNN
+F 2 "" H 800 10200 50  0001 C CNN
+F 3 "" H 800 10200 50  0001 C CNN
+	1    800  10200
 	1    0    0    -1
 $EndComp
@@
 	1350 9950 1150 9950
 Wire Wire Line
-	1150 9950 1150 10350
-Wire Wire Line
 	1050 9650 1050 9400
 $Comp
@@
 	1050 9400 1000 9400
 Connection ~ 1050 9400
-Wire Wire Line
-	3200 9750 3350 9750
-Text Label 3350 9750 0    50   ~ 0
+Text Label 3600 9750 0    50   ~ 0
 3.3V
 Text Label 14700 2800 2    50   ~ 0
@@
 Wire Notes Line
 	600  8650 8900 8650
+$Comp
+L formula:R_10K R29
+U 1 1 5BE079E8
+P 1200 10150
+F 0 "R29" V 1200 10150 50  0000 C CNN
+F 1 "R_10K" V 1300 10150 50  0000 C CNN
+F 2 "footprints:R_0805_OEM" H 1130 10150 50  0001 C CNN
+F 3 "http://www.bourns.com/data/global/pdfs/CRS.pdf" H 1280 10150 50  0001 C CNN
+F 4 "DK" H 1200 10150 60  0001 C CNN "MFN"
+F 5 "CRS0805-FX-1002ELFCT-ND" H 1200 10150 60  0001 C CNN "MPN"
+F 6 "https://www.digikey.com/products/en?keywords=CRS0805-FX-1002ELFCT-ND" H 1680 10550 60  0001 C CNN "PurchasingLink"
+	1    1200 10150
+	0    1    1    0
+$EndComp
+Wire Wire Line
+	1050 10150 800  10150
+Wire Wire Line
+	800  10150 800  10200
+Wire Wire Line
+	1150 9950 1150 10000
+Wire Wire Line
+	1150 10000 800  10000
+Wire Wire Line
+	800  10000 800  10150
+Connection ~ 800  10150
+$Comp
+L formula:R_10K R30
+U 1 1 5BE3C2D2
+P 1350 10500
+F 0 "R30" V 1350 10500 50  0000 C CNN
+F 1 "R_10K" V 1450 10500 50  0000 C CNN
+F 2 "footprints:R_0805_OEM" H 1280 10500 50  0001 C CNN
+F 3 "http://www.bourns.com/data/global/pdfs/CRS.pdf" H 1430 10500 50  0001 C CNN
+F 4 "DK" H 1350 10500 60  0001 C CNN "MFN"
+F 5 "CRS0805-FX-1002ELFCT-ND" H 1350 10500 60  0001 C CNN "MPN"
+F 6 "https://www.digikey.com/products/en?keywords=CRS0805-FX-1002ELFCT-ND" H 1830 10900 60  0001 C CNN "PurchasingLink"
+	1    1350 10500
+	-1   0    0    1
+$EndComp
+Wire Wire Line
+	1350 10650 1350 10700
+Wire Wire Line
+	1350 10700 1450 10700
+Text Label 1450 10700 0    50   ~ 0
+3.3V
+$Comp
+L formula:C_0.1uF C8
+U 1 1 5BE577AF
+P 3500 9900
+F 0 "C8" H 3615 9946 50  0000 L CNN
+F 1 "C_0.1uF" H 3615 9855 50  0000 L CNN
+F 2 "footprints:C_0805_OEM" H 3538 9750 50  0001 C CNN
+F 3 "http://datasheets.avx.com/X7RDielectric.pdf" H 3525 10000 50  0001 C CNN
+F 4 "DK" H 3500 9900 60  0001 C CNN "MFN"
+F 5 "478-3352-1-ND" H 3500 9900 60  0001 C CNN "MPN"
+F 6 "https://www.digikey.com/products/en?keywords=478-3352-1-ND" H 3925 10400 60  0001 C CNN "PurchasingLink"
+	1    3500 9900
+	1    0    0    -1
+$EndComp
+Wire Wire Line
+	3200 9750 3500 9750
+Connection ~ 3500 9750
+Wire Wire Line
+	3500 9750 3600 9750
+Wire Wire Line
+	3200 9950 3350 9950
+Wire Wire Line
+	3350 9950 3350 10050
+Wire Wire Line
+	3350 10050 3500 10050
+Wire Wire Line
+	3200 10150 3500 10150
+Wire Wire Line
+	3500 10150 3500 10250
+Wire Wire Line
+	3500 10050 3500 10150
+Connection ~ 3500 10050
+Connection ~ 3500 10150
 $EndSCHEMATC

Commit message: finished board
Parts:
- added C10, C9: C_0.1uF, footprints:C_0805_OEM, symbol formula:C_0.1uF
- F1: footprint Resistors_SMD:R_0402 -> footprints:R_0805_OEM
Connections:
- wire segments 210 -> 214
Changed lines of the file:
@@
 U 1 1 5BEEF940
 P 750 3350
-F 0 "J1" H 1200 4400 50  0000 L CNN
-F 1 "Conn_01x20_Female" H 1050 4500 50  0000 L CNN
+F 0 "J1" H 150 4300 50  0000 L CNN
+F 1 "Conn_01x20_Female" H 0   4400 50  0000 L CNN
 F 2 "footprints:Pin_Header_Straight_2x10" H 750 3350 50  0001 C CNN
 F 3 "~" H 750 3350 50  0001 C CNN
@@
 F 0 "F1" H 1660 1746 50  0000 L CNN
 F 1 "Fuse_1A" H 1660 1655 50  0000 L CNN
-F 2 "Resistors_SMD:R_0402" V 1530 1700 50  0001 C CNN
+F 2 "footprints:R_0805_OEM" V 1530 1700 50  0001 C CNN
 F 3 "https://industrial.panasonic.com/cdbs/www-data/pdf/AFA0000/AFA0000C7.pdf" H 1600 1700 50  0001 C CNN
 	1    1600 1700
-	1    0    0    -1
+	-1   0    0    1
 $EndComp
 Text Notes 1450 9050 0    118  ~ 0
@@
 $EndComp
 Wire Wire Line
-	5450 1300 5350 1300
-Wire Wire Line
-	5350 1300 5350 1150
+	5450 1300 5400 1300
 $Comp
 L power:VCC #PWR022
@@
 Wire Wire Line
 	6050 1300 6100 1300
-Text Label 6100 1300 0    50   ~ 0
+Text Label 6200 1300 0    50   ~ 0
 3.3V
 Wire Wire Line
@@
 Connection ~ 3500 10050
 Connection ~ 3500 10150
+$Comp
+L formula:C_0.1uF C9
+U 1 1 5BE1A86E
+P 5400 1450
+F 0 "C9" H 5200 1450 50  0000 L CNN
+F 1 "C_0.1uF" H 5100 1350 50  0000 L CNN
+F 2 "footprints:C_0805_OEM" H 5438 1300 50  0001 C CNN
+F 3 "http://datasheets.avx.com/X7RDielectric.pdf" H 5425 1550 50  0001 C CNN
+F 4 "DK" H 5400 1450 60  0001 C CNN "MFN"
+F 5 "478-3352-1-ND" H 5400 1450 60  0001 C CNN "MPN"
+F 6 "https://www.digikey.com/products/en?keywords=478-3352-1-ND" H 5825 1950 60  0001 C CNN "PurchasingLink"
+	1    5400 1450
+	1    0    0    -1
+$EndComp
+$Comp
+L formula:C_0.1uF C10
+U 1 1 5BE1A926
+P 6100 1450
+F 0 "C10" H 6200 1450 50  0000 L CNN
+F 1 "C_0.1uF" H 6100 1350 50  0000 L CNN
+F 2 "footprints:C_0805_OEM" H 6138 1300 50  0001 C CNN
+F 3 "http://datasheets.avx.com/X7RDielectric.pdf" H 6125 1550 50  0001 C CNN
+F 4 "DK" H 6100 1450 60  0001 C CNN "MFN"
+F 5 "478-3352-1-ND" H 6100 1450 60  0001 C CNN "MPN"
+F 6 "https://www.digikey.com/products/en?keywords=478-3352-1-ND" H 6525 1950 60  0001 C CNN "PurchasingLink"
+	1    6100 1450
+	1    0    0    -1
+$EndComp
+Wire Wire Line
+	5400 1300 5350 1300
+Wire Wire Line
+	5350 1300 5350 1150
+Connection ~ 5400 1300
+Wire Wire Line
+	6100 1300 6200 1300
+Connection ~ 6100 1300
+Wire Wire Line
+	6100 1600 5750 1600
+Connection ~ 5750 1600
+Wire Wire Line
+	5400 1600 5750 1600
 $EndSCHEMATC

Commit message: Added a LED circuit
Parts:
- added D3: D_Photo, symbol Device:D_Photo
- added R27: R_1K, footprints:R_0805_OEM, symbol formula:R_1K
- P1: symbol formula:CONN_02X03 -> circuit-rescue:CONN_02X03-formula
Connections:
- net labels added: +3.3V, Measurement_Point
- wire segments 214 -> 217
Other:
- note added: "Light Intensity Detection"
Changed lines of the file:
@@
 	14400 3000 14400 3100
 $Comp
-L formula:CONN_02X03 P1
+L circuit-rescue:CONN_02X03-formula P1
 U 1 1 5BCC9EE8
 P 2700 2800
@@
 	1    0    0    -1
 $EndComp
-Wire Wire Line
-	14700 6000 14700 5900
-Wire Wire Line
-	14700 5900 14700 5800
-Connection ~ 14700 5900
-Wire Wire Line
-	14700 5800 14700 5600
-Connection ~ 14700 5800
 $Comp
 L power:VCC #PWR046
@@
 Wire Wire Line
 	14700 6300 14850 6300
-Connection ~ 14700 6300
 Wire Wire Line
 	14700 6200 15300 6200
@@
 Wire Wire Line
 	12850 6000 12850 6200
-Connection ~ 13450 6000
 Connection ~ 12850 6200
 Text Label 14700 1600 2    50   ~ 0
@@
 Wire Wire Line
 	3850 6000 3950 6000
-Connection ~ 3850 6000
 Wire Wire Line
 	3300 6400 3300 6450
@@
 Wire Wire Line
 	7850 5950 7950 5950
-Connection ~ 7850 5950
 Wire Wire Line
 	7300 6350 7300 6400
@@
 Wire Wire Line
 	3850 7850 3950 7850
-Connection ~ 3850 7850
 Wire Wire Line
 	3300 8250 3300 8300
@@
 Wire Wire Line
 	7800 7850 7900 7850
-Connection ~ 7800 7850
 Wire Wire Line
 	7250 8250 7250 8300
@@
 Wire Wire Line
 	5400 1600 5750 1600
+Wire Wire Line
+	14700 5600 14700 6000
+$Comp
+L Device:D_Photo D3
+U 1 1 5C13FD7A
+P 6050 9800
+F 0 "D3" H 6000 9584 50  0000 C CNN
+F 1 "D_Photo" H 6000 9675 50  0000 C CNN
+F 2 "" H 6000 9800 50  0001 C CNN
+F 3 "~" H 6000 9800 50  0001 C CNN
+	1    6050 9800
+	-1   0    0    1
+$EndComp
+$Comp
+L power:+3.3V #PWR05
+U 1 1 5C13FF5C
+P 5500 9650
+F 0 "#PWR05" H 5500 9500 50  0001 C CNN
+F 1 "+3.3V" H 5515 9823 50  0000 C CNN
+F 2 "" H 5500 9650 50  0001 C CNN
+F 3 "" H 5500 9650 50  0001 C CNN
+	1    5500 9650
+	1    0    0    -1
+$EndComp
+$Comp
+L formula:R_1K R27
+U 1 1 5C14007D
+P 6650 10150
+F 0 "R27" H 6720 10196 50  0000 L CNN
+F 1 "R_1K" H 6720 10105 50  0000 L CNN
+F 2 "footprints:R_0805_OEM" H 6580 10150 50  0001 C CNN
+F 3 "https://www.seielect.com/Catalog/SEI-rncp.pdf" H 6730 10150 50  0001 C CNN
+F 4 "DK" H 6650 10150 60  0001 C CNN "MFN"
+F 5 "RNCP0805FTD1K00CT-ND" H 6650 10150 60  0001 C CNN "MPN"
+F 6 "https://www.digikey.com/products/en?keywords=RNCP0805FTD1K00CT-ND" H 7130 10550 60  0001 C CNN "PurchasingLink"
+	1    6650 10150
+	1    0    0    -1
+$EndComp
+$Comp
+L power:GND #PWR053
+U 1 1 5C140200
+P 6650 10300
+F 0 "#PWR053" H 6650 10050 50  0001 C CNN
+F 1 "GND" H 6655 10127 50  0000 C CNN
+F 2 "" H 6650 10300 50  0001 C CNN
+F 3 "" H 6650 10300 50  0001 C CNN
+	1    6650 10300
+	1    0    0    -1
+$EndComp
+Text GLabel 7050 9800 2    59   Input ~ 0
+Measurement_Point
+Wire Wire Line
+	5500 9650 5500 9800
+Wire Wire Line
+	5500 9800 5950 9800
+Wire Wire Line
+	6250 9800 6650 9800
+Wire Wire Line
+	6650 9800 6650 10000
+Wire Wire Line
+	6650 9800 7050 9800
+Connection ~ 6650 9800
+Text Notes 7700 9000 2    118  ~ 0
+Light Intensity Detection
 $EndSCHEMATC
