File: beacon/beacon.sch (KiCad schematic (older format))
At the start: 6 parts, among them J1 Conn_01x03_Female, SW1 SW_Push, U1 ATtiny45-20PU

Commit message: Added a LED circuit
Parts:
- R1: symbol formula:R_10K -> beacon-rescue:R_10K-formula
- R2: symbol formula:R_200 -> beacon-rescue:R_200-formula
Changed lines of the file:
@@
 $EndComp
 $Comp
-L formula:R_200 R2
+L beacon-rescue:R_200-formula R2
 U 1 1 5BDF762D
 P 5850 3450
@@
 PB2
 $Comp
-L formula:R_10K R1
+L beacon-rescue:R_10K-formula R1
 U 1 1 5BDF8DC0
 P 2600 3900
